File: dru-template/dru-template.kicad_pcb (KiCad board)
At the start: 2 copper layers, 0 parts

Commit message: Update dru-template.kicad_pcb
Other:
- net class class1 added: clearance 0.7, trace_width 0.8, via_dia 0.9, via_drill 0.5
- net class class2 added: clearance 0.5, trace_width 0.5, via_dia 0.6, via_drill 0.3
- net class class3 added: clearance 0.35, trace_width 0.5, via_dia 0.6, via_drill 0.3
- net class class4 added: clearance 0.25, trace_width 0.23, via_dia 0.6, via_drill 0.3
- net class クラス1 removed
- net class クラス2 removed
- net class クラス3 removed
- net class クラス4 removed
Changed lines of the file:
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@@
     (uvia_drill 0.1)
   )
-  (net_class クラス1 ""
+  (net_class class1 ""
     (clearance 0.7)
     (trace_width 0.8)
@@
     (uvia_drill 0.1)
   )
-  (net_class クラス2 ""
+  (net_class class2 ""
     (clearance 0.5)
     (trace_width 0.5)
@@
     (uvia_drill 0.1)
   )
-  (net_class クラス3 ""
+  (net_class class3 ""
     (clearance 0.35)
     (trace_width 0.5)
@@
     (uvia_drill 0.1)
   )
-  (net_class クラス4 ""
+  (net_class class4 ""
     (clearance 0.25)
     (trace_width 0.23)
